Commit message: Small fixes on Go2

File: src/robot_properties_solo/resources/xacro/solo/leg.xacro (robot description, xacro)
@@ -50,5 +50,5 @@
                     <origin xyz="0.0 0 0" rpy="0 0 0" />
                     <geometry>
-                        <mesh filename="package://robot_properties_solo/resources/meshes/${mesh_ext}/solo12/solo12_hip_fe_fl.${mesh_ext}"/>
+                        <mesh filename="package://robot_properties_solo/resources/meshes/solo/${mesh_ext}/solo12/solo12_hip_fe_fl.${mesh_ext}"/>
                     </geometry>
                 </xacro:if>
@@ -56,5 +56,5 @@
                     <origin xyz="-0.0 0 0" rpy="0 0 0" />
                     <geometry>
-                        <mesh filename="package://robot_properties_solo/resources/meshes/${mesh_ext}/solo12/solo12_hip_fe_hl.${mesh_ext}"/>
+                        <mesh filename="package://robot_properties_solo/resources/meshes/solo/${mesh_ext}/solo12/solo12_hip_fe_hl.${mesh_ext}"/>
                     </geometry>
                 </xacro:unless>
@@ -64,5 +64,5 @@
                     <origin xyz="0.0 0 0" rpy="0 0 0" />
                     <geometry>
-                        <mesh filename="package://robot_properties_solo/resources/meshes/${mesh_ext}/solo12/solo12_hip_fe_fr.${mesh_ext}"/>
+                        <mesh filename="package://robot_properties_solo/resources/meshes/solo/${mesh_ext}/solo12/solo12_hip_fe_fr.${mesh_ext}"/>
                     </geometry>
                 </xacro:if>
@@ -70,5 +70,5 @@
                     <origin xyz="-0.0 0 0" rpy="0 0 0" />
                     <geometry>
-                        <mesh filename="package://robot_properties_solo/resources/meshes/${mesh_ext}/solo12/solo12_hip_fe_hr.${mesh_ext}"/>
+                        <mesh filename="package://robot_properties_solo/resources/meshes/solo/${mesh_ext}/solo12/solo12_hip_fe_hr.${mesh_ext}"/>
                     </geometry>
                 </xacro:unless>
@@ -84,5 +84,5 @@
                     <origin xyz="0.0 0 0" rpy="0 0 0" />
                     <geometry>
-                        <mesh filename="package://robot_properties_solo/resources/meshes/${mesh_ext}/solo12/solo12_hip_fe_fl.${mesh_ext}"/>
+                        <mesh filename="package://robot_properties_solo/resources/meshes/solo/${mesh_ext}/solo12/solo12_hip_fe_fl.${mesh_ext}"/>
                     </geometry>
                 </xacro:if>
@@ -90,5 +90,5 @@
                     <origin xyz="-0.0 0 0" rpy="0 0 0" />
                     <geometry>
-                        <mesh filename="package://robot_properties_solo/resources/meshes/${mesh_ext}/solo12/solo12_hip_fe_hl.${mesh_ext}"/>
+                        <mesh filename="package://robot_properties_solo/resources/meshes/solo/${mesh_ext}/solo12/solo12_hip_fe_hl.${mesh_ext}"/>
                     </geometry>
                 </xacro:unless>
@@ -98,5 +98,5 @@
                     <origin xyz="0.0 0 0" rpy="0 0 0" />
                     <geometry>
-                        <mesh filename="package://robot_properties_solo/resources/meshes/${mesh_ext}/solo12/solo12_hip_fe_fr.${mesh_ext}"/>
+                        <mesh filename="package://robot_properties_solo/resources/meshes/solo/${mesh_ext}/solo12/solo12_hip_fe_fr.${mesh_ext}"/>
                     </geometry>
                 </xacro:if>
@@ -104,5 +104,5 @@
                     <origin xyz="-0.0 0 0" rpy="0 0 0" />
                     <geometry>
-                        <mesh filename="package://robot_properties_solo/resources/meshes/${mesh_ext}/solo12/solo12_hip_fe_hr.${mesh_ext}"/>
+                        <mesh filename="package://robot_properties_solo/resources/meshes/solo/${mesh_ext}/solo12/solo12_hip_fe_hr.${mesh_ext}"/>
                     </geometry>
                 </xacro:unless>
@@ -231,8 +231,8 @@
         <geometry>
           <xacro:unless value="${is_right}">
-            <mesh filename="package://robot_properties_solo/resources/meshes/${mesh_ext}/without_foot/solo_upper_leg_left_side.${mesh_ext}"/>
-          </xacro:unless>
-          <xacro:if value="${is_right}">
-            <mesh filename="package://robot_properties_solo/resources/meshes/${mesh_ext}/without_foot/solo_upper_leg_right_side.${mesh_ext}"/>
+            <mesh filename="package://robot_properties_solo/resources/meshes/solo/${mesh_ext}/without_foot/solo_upper_leg_left_side.${mesh_ext}"/>
+          </xacro:unless>
+          <xacro:if value="${is_right}">
+            <mesh filename="package://robot_properties_solo/resources/meshes/solo/${mesh_ext}/without_foot/solo_upper_leg_right_side.${mesh_ext}"/>
           </xacro:if>
         </geometry>
@@ -246,8 +246,8 @@
         <geometry>
           <xacro:unless value="${is_right}">
-            <mesh filename="package://robot_properties_solo/resources/meshes/${mesh_ext}/without_foot/solo_upper_leg_left_side.${mesh_ext}"/>
-          </xacro:unless>
-          <xacro:if value="${is_right}">
-            <mesh filename="package://robot_properties_solo/resources/meshes/${mesh_ext}/without_foot/solo_upper_leg_right_side.${mesh_ext}"/>
+            <mesh filename="package://robot_properties_solo/resources/meshes/solo/${mesh_ext}/without_foot/solo_upper_leg_left_side.${mesh_ext}"/>
+          </xacro:unless>
+          <xacro:if value="${is_right}">
+            <mesh filename="package://robot_properties_solo/resources/meshes/solo/${mesh_ext}/without_foot/solo_upper_leg_right_side.${mesh_ext}"/>
           </xacro:if>
         </geometry>
@@ -316,8 +316,8 @@
         <geometry>
           <xacro:unless value="${is_right}">
-            <mesh filename="package://robot_properties_solo/resources/meshes/${mesh_ext}/without_foot/solo_lower_leg_v2_left_side.${mesh_ext}"/>
-          </xacro:unless>
-          <xacro:if value="${is_right}">
-            <mesh filename="package://robot_properties_solo/resources/meshes/${mesh_ext}/without_foot/solo_lower_leg_v2_right_side.${mesh_ext}"/>
+            <mesh filename="package://robot_properties_solo/resources/meshes/solo/${mesh_ext}/without_foot/solo_lower_leg_v2_left_side.${mesh_ext}"/>
+          </xacro:unless>
+          <xacro:if value="${is_right}">
+            <mesh filename="package://robot_properties_solo/resources/meshes/solo/${mesh_ext}/without_foot/solo_lower_leg_v2_right_side.${mesh_ext}"/>
           </xacro:if>
         </geometry>
@@ -331,8 +331,8 @@
         <geometry>
           <xacro:unless value="${is_right}">
-            <mesh filename="package://robot_properties_solo/resources/meshes/${mesh_ext}/without_foot/solo_lower_leg_v2_left_side.${mesh_ext}"/>
-          </xacro:unless>
-          <xacro:if value="${is_right}">
-            <mesh filename="package://robot_properties_solo/resources/meshes/${mesh_ext}/without_foot/solo_lower_leg_v2_right_side.${mesh_ext}"/>
+            <mesh filename="package://robot_properties_solo/resources/meshes/solo/${mesh_ext}/without_foot/solo_lower_leg_v2_left_side.${mesh_ext}"/>
+          </xacro:unless>
+          <xacro:if value="${is_right}">
+            <mesh filename="package://robot_properties_solo/resources/meshes/solo/${mesh_ext}/without_foot/solo_lower_leg_v2_right_side.${mesh_ext}"/>
           </xacro:if>
         </geometry>

File: src/robot_properties_solo/resources/xacro/solo12.urdf.xacro (robot description, xacro)
@@ -25,5 +25,5 @@
         <origin xyz="0 0 0" rpy="0 0 0" />
         <geometry>
-          <mesh filename="package://robot_properties_solo/resources/meshes/${mesh_ext}/solo12/solo_12_base.${mesh_ext}"/>
+          <mesh filename="package://robot_properties_solo/resources/meshes/solo/${mesh_ext}/solo12/solo_12_base.${mesh_ext}"/>
         </geometry>
         <material name="${color_name}">
@@ -35,5 +35,5 @@
         <origin xyz="0 0 0" rpy="0 0 0" />
         <geometry>
-          <mesh filename="package://robot_properties_solo/resources/meshes/${mesh_ext}/solo12/solo_12_base.${mesh_ext}"/>
+          <mesh filename="package://robot_properties_solo/resources/meshes/solo/${mesh_ext}/solo12/solo_12_base.${mesh_ext}"/>
         </geometry>
         <material name="${color_name}">
