Commit message: Added go2

File: src/robot_properties_solo/resources/mjcf/solo12.mjcf.xacro (robot description, xacro)
@@ -7,5 +7,5 @@
         <geom solref="0.005 20" solimp= "0.99 0.999 0.002 0.5 2"/>
     </default>
-    <compiler angle="radian" meshdir="$(arg resources_dir)/meshes/stl/solo12/" autolimits="true"/>
+    <compiler angle="radian" meshdir="$(arg resources_dir)/meshes/solo/stl/solo12/" autolimits="true"/>
     <asset>
         <texture name="grid" type="2d" builtin="checker" rgb1=".1 .2 .3"
@@ -37,8 +37,8 @@
         <body name="base_link" pos="0 0 0.4" euler="0 0 0">
             <joint name="free_joint" type="free"/>
-            <inertial mass="1.25123725" pos="0 0 0" fullinertia="0.00266220 0.01388510 0.01605370 -0.00003684 -0.00001716 -0.00000009"/>
+            <inertial mass="1.52123725" pos="0 0 0" fullinertia="0.00266220 0.01388510 0.01605370 -0.00003684 -0.00001716 -0.00000009"/>
             <geom type="mesh" mesh="solo_12_base"/>
             <body name="FL_SHOULDER" pos="0.2141 0.0875 0">
-                <joint name="FL_HAA" type="hinge" axis="1 0 0" range="-0.9 0.9" damping="0.009" frictionloss="0.003"/>
+                <joint name="FL_HAA" type="hinge" axis="1 0 0" range="-1.0 1.0" damping="0.009" frictionloss="0.003"/>
                 <geom type="mesh" mesh="solo12_hip_fe_fl"/>
                 <inertial mass="0.14196048" pos="-0.09407251 -0.00438935 0.00001384" fullinertia="0.00002802 0.00038264 0.00038050 0.00003687 -0.00000009 0.00000000"/>
@@ -56,5 +56,5 @@
             </body>
             <body name="FR_SHOULDER" pos="0.2141 -0.08750 0">
-                <joint name="FR_HAA" type="hinge" axis="1 0 0" range="-0.9 0.9" damping="0.009" frictionloss="0.003"/>
+                <joint name="FR_HAA" type="hinge" axis="1 0 0" range="-1 1" damping="0.009" frictionloss="0.003"/>
                 <geom type="mesh" mesh="solo12_hip_fe_fr"/>
                 <inertial mass="0.14196048" pos="-0.09407251 0.00438935 -0.00001384" fullinertia="0.00002802 0.00038264 0.00038050 -0.00003687 0.00000009 0.00000000"/>
@@ -72,5 +72,5 @@
             </body>
             <body name="HL_SHOULDER" pos="-0.2141 0.08750000000000001 0">
-                <joint name="HL_HAA" type="hinge" axis="1 0 0" range="-0.9 0.9" damping="0.009" frictionloss="0.003"/>
+                <joint name="HL_HAA" type="hinge" axis="1 0 0" range="-1 1" damping="0.009" frictionloss="0.003"/>
                 <geom type="mesh" mesh="solo12_hip_fe_hl"/>
                 <inertial mass="0.14196048" pos="0.09407251 -0.00438935 -0.00001384" fullinertia="0.00002802 0.00038264 0.00038050 -0.00003687 -0.00000009 0.00000000"/>
@@ -88,5 +88,5 @@
             </body>
             <body name="HR_SHOULDER" pos="-0.2141 -0.08750000000000001 0">
-                <joint name="HR_HAA" type="hinge" axis="1 0 0" range="-0.9 0.9" damping="0.009" frictionloss="0.003"/>
+                <joint name="HR_HAA" type="hinge" axis="1 0 0" range="-1 1" damping="0.009" frictionloss="0.003"/>
                 <geom type="mesh" mesh="solo12_hip_fe_hr"/>
                 <inertial mass="0.14196048" pos="0.09407251 0.00438935 0.00001384" fullinertia="0.00002802 0.00038264 0.00038050 0.00003687 0.00000009 0.00000000"/>

File: src/robot_properties_solo/resources/xacro/solo12.urdf.xacro (robot description, xacro)
@@ -13,6 +13,6 @@
     <!-- BASE LINK INERTIAL -->
     <inertial>
-        <origin xyz="-0.00082966 0.00000105 -0.00060210" rpy="0 0 0" />
-        <mass value="1.25123725"/>
+        <origin xyz="-0.02 0.00 .0" rpy="0 0 0" />
+        <mass value="1.62123725"/>
         <!-- The base is extremely symmetrical. -->
         <inertia ixx="0.00266220" ixy="-0.00003684" ixz="-0.00001716"
@@ -48,5 +48,5 @@
   </link> <!-- END BASE LINK -->
   <!-- Include the legs -->
-  <xacro:include filename="leg.xacro"/>
+  <xacro:include filename="solo/leg.xacro"/>
   <!-- Include the front left leg -->
   <xacro:leg

File: src/robot_properties_solo/resources/xacro/solo13.urdf.xacro (robot description, xacro)
@@ -86,5 +86,5 @@
   </joint>
   <!-- Include the legs -->
-  <xacro:include filename="leg.xacro"/>
+  <xacro:include filename="solo/leg.xacro"/>
   <!-- Include the front left leg -->
   <xacro:leg prefix="FL" parent="base_link" is_front="true" is_right="false" has_side_motion="true" mesh_ext="${mesh_ext}" color_name="${color_name}" color="${color}" opacity="${opacity}"/>

File: src/robot_properties_solo/resources/xacro/solo6.urdf.xacro (robot description, xacro)
@@ -48,5 +48,5 @@
   </link> <!-- END BASE LINK -->
   <!-- Include the legs -->
-  <xacro:include filename="leg.xacro"/>
+  <xacro:include filename="solo/leg.xacro"/>
   <!-- Include the front left leg -->
   <xacro:leg

File: src/robot_properties_solo/resources/xacro/solo8.urdf.xacro (robot description, xacro)
@@ -48,5 +48,5 @@
   </link> <!-- END BASE LINK -->
   <!-- Include the legs -->
-  <xacro:include filename="leg.xacro"/>
+  <xacro:include filename="solo/leg.xacro"/>
   <!-- Include the front left leg -->
   <xacro:leg

Commit message: Added anymal

File: src/robot_properties_solo/resources/mjcf/solo12.mjcf.xacro (robot description, xacro)
@@ -37,5 +37,5 @@
         <body name="base_link" pos="0 0 0.4" euler="0 0 0">
             <joint name="free_joint" type="free"/>
-            <inertial mass="1.52123725" pos="0 0 0" fullinertia="0.00266220 0.01388510 0.01605370 -0.00003684 -0.00001716 -0.00000009"/>
+            <inertial mass="1.62123725" pos="0 0 0" fullinertia="0.00266220 0.01388510 0.01605370 -0.00003684 -0.00001716 -0.00000009"/>
             <geom type="mesh" mesh="solo_12_base"/>
             <body name="FL_SHOULDER" pos="0.2141 0.0875 0">
